File: pcb/Anemometro/pcbanemometro/Placa ANEMOMETRO.kicad_sch (KiCad schematic)
At the start: 14 parts, among them J1 Conn_01x03, J2 Conn_01x03, U1 TL082

Commit message: se readaptaron y revisaron las PCBs, listas para imprimir
Parts:
- C3: footprint Capacitor_THT:C_Radial_D5.0mm_H7.0mm_P2.00mm -> Capacitor_THT:C_Radial_D8.0mm_H7.0mm_P3.50mm
- J1: value Conn_01x03 -> SS41
- J2: value Conn_01x03 -> ToMother
- R1, R2, R3: footprint Resistor_THT:R_Axial_DIN0207_L6.3mm_D2.5mm_P7.62mm_Horizontal -> Resistor_THT:R_Axial_DIN0207_L6.3mm_D2.5mm_P10.16mm_Horizontal
Connections:
- net D_hall: now also J2.3 (Pin_3); no longer J2.2 (Pin_2)
- net GND_G1: now also J2.2 (Pin_2); no longer J2.3 (Pin_3)
Other:
- moved on the sheet: J2
Changed lines of the file:
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@@
 	(wire
 		(pts
-			(xy 234.95 66.04) (xy 231.14 66.04)
+			(xy 147.32 44.45) (xy 143.51 44.45)
 		)
 		(stroke
@@
 	(wire
 		(pts
-			(xy 234.95 69.85) (xy 232.41 69.85)
+			(xy 147.32 46.99) (xy 143.51 46.99)
 		)
 		(stroke
@@
 	(wire
 		(pts
-			(xy 234.95 68.58) (xy 234.95 69.85)
-		)
-		(stroke
-			(width 0)
-			(type default)
-		)
-	)
-	(wire
-		(pts
 			(xy 179.07 90.17) (xy 208.28 90.17)
 		)
@@
 	(wire
 		(pts
-			(xy 234.95 63.5) (xy 234.95 43.18)
+			(xy 147.32 41.91) (xy 147.32 36.83)
 		)
 		(stroke
@@
 	(global_label "GND_G1"
 		(shape input)
-		(at 232.41 69.85 180)
+		(at 143.51 44.45 180)
 		(fields_autoplaced yes)
 		(effects
@@
 		)
 		(property "Intersheetrefs" "${INTERSHEET_REFS}"
-			(at 222.1072 69.85 0)
+			(at 133.2072 44.45 0)
 			(effects
 				(font
@@
 	(global_label "D_hall"
 		(shape input)
-		(at 231.14 66.04 180)
+		(at 143.51 46.99 180)
 		(fields_autoplaced yes)
 		(effects
@@
 		)
 		(property "Intersheetrefs" "${INTERSHEET_REFS}"
-			(at 222.2888 66.04 0)
+			(at 134.6588 46.99 0)
 			(effects
 				(font
@@
 	(symbol
 		(lib_id "power:VD")
-		(at 234.95 43.18 0)
+		(at 147.32 36.83 0)
 		(unit 1)
 		(exclude_from_sim no)
@@
 		(fields_autoplaced yes)
 		(property "Reference" "#PWR07"
-			(at 234.95 46.99 0)
+			(at 147.32 40.64 0)
 			(effects
 				(font
@@
 		)
 		(property "Value" "3.3V"
-			(at 234.95 38.1 0)
+			(at 147.32 31.75 0)
 			(effects
 				(font
@@
 		)
 		(property "Footprint" ""
-			(at 234.95 43.18 0)
+			(at 147.32 36.83 0)
 			(effects
 				(font
@@
 		)
 		(property "Datasheet" ""
-			(at 234.95 43.18 0)
+			(at 147.32 36.83 0)
 			(effects
 				(font
@@
 		)
 		(property "Description" "Power symbol creates a global label with name \"VD\""
-			(at 234.95 43.18 0)
+			(at 147.32 36.83 0)
 			(effects
 				(font
@@
 			)
 		)
-		(property "Footprint" "Resistor_THT:R_Axial_DIN0207_L6.3mm_D2.5mm_P7.62mm_Horizontal"
+		(property "Footprint" "Resistor_THT:R_Axial_DIN0207_L6.3mm_D2.5mm_P10.16mm_Horizontal"
 			(at 60.706 76.454 90)
 			(effects
@@
 			)
 		)
-		(property "Footprint" "Resistor_THT:R_Axial_DIN0207_L6.3mm_D2.5mm_P7.62mm_Horizontal"
+		(property "Footprint" "Resistor_THT:R_Axial_DIN0207_L6.3mm_D2.5mm_P10.16mm_Horizontal"
 			(at 73.406 53.594 90)
 			(effects
@@
 			)
 		)
-		(property "Value" "Conn_01x03"
+		(property "Value" "SS41"
 			(at 43.18 69.85 0)
 			(effects
@@
 	(symbol
 		(lib_id "Connector_Generic:Conn_01x03")
-		(at 240.03 66.04 0)
+		(at 152.4 44.45 0)
 		(unit 1)
 		(exclude_from_sim no)
@@
 		(fields_autoplaced yes)
 		(property "Reference" "J2"
-			(at 242.57 64.7699 0)
-			(effects
-				(font
-					(size 1.27 1.27)
-				)
-				(justify left)
-			)
-		)
-		(property "Value" "Conn_01x03"
-			(at 242.57 67.3099 0)
+			(at 154.94 43.1799 0)
+			(effects
+				(font
+					(size 1.27 1.27)
+				)
+				(justify left)
+			)
+		)
+		(property "Value" "ToMother"
+			(at 154.94 45.7199 0)
 			(effects
 				(font
@@
 		)
 		(property "Footprint" "Connector_PinHeader_2.54mm:PinHeader_1x03_P2.54mm_Vertical"
-			(at 240.03 66.04 0)
+			(at 152.4 44.45 0)
 			(effects
 				(font
@@
 		)
 		(property "Datasheet" "~"
-			(at 240.03 66.04 0)
+			(at 152.4 44.45 0)
 			(effects
 				(font
@@
 		)
 		(property "Description" "Generic connector, single row, 01x03, script generated (kicad-library-utils/schlib/autogen/connector/)"
-			(at 240.03 66.04 0)
+			(at 152.4 44.45 0)
 			(effects
 				(font
@@
 			)
 		)
-		(property "Footprint" "Capacitor_THT:C_Radial_D5.0mm_H7.0mm_P2.00mm"
+		(property "Footprint" "Capacitor_THT:C_Radial_D8.0mm_H7.0mm_P3.50mm"
 			(at 208.28 66.04 0)
 			(effects
@@
 			)
 		)
-		(property "Footprint" "Resistor_THT:R_Axial_DIN0207_L6.3mm_D2.5mm_P7.62mm_Horizontal"
+		(property "Footprint" "Resistor_THT:R_Axial_DIN0207_L6.3mm_D2.5mm_P10.16mm_Horizontal"
 			(at 119.126 53.594 90)
 			(effects
